Commit message: added new methods and services

File: quadrotor_controller/urdf/quadrotor_with_asus_with_2lasers.urdf.xacro (robot description, xacro)
@@ -14,5 +14,5 @@
     <xacro:include filename="$(find hector_sensors_description)/urdf/asus_camera.urdf.xacro" />
     <xacro:asus_camera name="camera" parent="base_link">
-      <origin xyz="0.1 0.0 -0.03" rpy="0 0 0"/>
+      <origin xyz="0.1 0.0 -0.03" rpy="0 ${M_PI/9} 0"/>
     </xacro:asus_camera>
         <!-- Asus Xiton Live Pro -->
