Commit message: made changes on quadrotor and adaptation on semantic map

File: quadrotor_controller/urdf/quadrotor_base.urdf.xacro (robot description, xacro)
@@ -25,5 +25,5 @@
     </link>
     <!-- Sonar height sensor -->
-    <xacro:sonar_sensor name="sonar" parent="base_link" ros_topic="sonar_height" update_rate="10" min_range="0.03" max_range="8.0" field_of_view="3" ray_count="3"> <!-- field of view ${40*pi/180} -->
+    <xacro:sonar_sensor name="sonar" parent="base_link" ros_topic="sonar_height" update_rate="10" min_range="0.03" max_range="8.0" field_of_view="3" ray_count="3"> <!-- field of view  ${40*pi/180} -->
       <origin xyz="-0.16 0.0 -0.012" rpy="0 ${90*pi/180} 0"/>
     </xacro:sonar_sensor>

File: quadrotor_controller/urdf/quadrotor_with_kinect.urdf.xacro (robot description, xacro)
@@ -9,5 +9,6 @@
     <xacro:include filename="$(find quadrotor_controller)/urdf/kinect_camera.urdf.xacro" />
     <xacro:kinect_camera name="camera" parent="base_link">
-      <origin xyz="0.1 0.0 -0.05" rpy="0 1.4 0"/>
+      <origin xyz="0.1 0.0 -0.04" rpy="0 0 0"/>
+<!-- "0.05 0.0 -0.06" "0 1.4 0" -->
     </xacro:kinect_camera>
 </robot>
