Commit message: changed kinect rotation

File: quadrotor_controller/urdf/quadrotor_with_kinect.urdf.xacro (robot description, xacro)
@@ -9,5 +9,5 @@
     <xacro:include filename="$(find quadrotor_controller)/urdf/kinect_camera.urdf.xacro" />
     <xacro:kinect_camera name="camera" parent="base_link">
-      <origin xyz="0.1 0.0 -0.04" rpy="0 0 0"/>
+      <origin xyz="0.1 0.0 -0.06" rpy="0 0.2 0"/>
 <!-- "0.05 0.0 -0.06" "0 1.4 0" -->
     </xacro:kinect_camera>
