Commit message: change cam-position

File: quadrotor_controller/urdf/asus_camera.urdf.xacro (robot description, xacro)
@@ -75,11 +75,11 @@
       <gazebo reference="${name}_depth_frame">
         <sensor type="depth" name="${name}">
-          <update_rate>80</update_rate>
+          <update_rate>100</update_rate>
           <camera>
             <horizontal_fov>${62.8 * M_PI/180.0}</horizontal_fov>
             <image>
               <format>R8G8B8</format>
-              <width>1040</width>
-              <height>880</height>
+              <width>2840</width>
+              <height>980</height>
             </image>
             <clip>

File: quadrotor_controller/urdf/quadrotor_with_asus_with_2lasers.urdf.xacro (robot description, xacro)
@@ -7,13 +7,14 @@
     <xacro:quadrotor_base_macro />
     <!-- Hokuyo UTM-30LX mounted upside down below the quadrotor body -->
-    <xacro:include filename="$(find quadrotor_controller)/urdf/hokuyo_utm30lx.urdf.xacro" />
+    <!--xacro:include filename="$(find quadrotor_controller)/urdf/hokuyo_utm30lx.urdf.xacro" />
     <xacro:hokuyo_utm30lx name="laser0" parent="base_link" ros_topic="scan" update_rate="80" ray_count="3081" min_angle="-285" max_angle="285">
       <origin xyz="0.0 0.0 -0.097" rpy="${M_PI} 0 0"/>
-    </xacro:hokuyo_utm30lx>
+    </xacro:hokuyo_utm30lx-->
     <!-- Asus Xiton Live Pro -->
     <xacro:include filename="$(find quadrotor_controller)/urdf/asus_camera.urdf.xacro" />
     <xacro:asus_camera name="camera" parent="base_link">
-      <origin xyz="0.1 0.0 -0.03" rpy="0 ${M_PI/9} 0"/>
+      <origin xyz="0.1 0.0 -0.05" rpy="0 1.5 0"/>
     </xacro:asus_camera>
+    <!--${M_PI/9}-->
         <!-- Asus Xiton Live Pro -->
     <!--xacro:include filename="$(find hector_sensors_description)/urdf/asus_camera.urdf.xacro" />

Commit message: added quadrotor

File: quadrotor_controller/urdf/asus_camera.urdf.xacro (robot description, xacro)
@@ -86,5 +86,5 @@
             <clip>
               <near>1</near>
-              <far>100</far>
+              <far>30</far>
             </clip>
           </camera>

File: quadrotor_controller/urdf/kinect_camera.urdf.xacro (robot description, xacro)
@@ -61,8 +61,8 @@
             <image>
               <format>R8G8B8</format>
-	      <!--width>640</width>
-	      <height>480</height-->
-              <width>1540</width>
-              <height>3580</height>
+	      <width>1540</width>
+	      <height>3580</height>
+              <!--width>1540</width>
+              <height>3580</height-->
             </image>
             <clip>

File: quadrotor_controller/urdf/quadrotor_with_kinect.urdf.xacro (robot description, xacro)
@@ -12,3 +12,8 @@
 <!-- "0.05 0.0 -0.06" "0 1.4 0" -->
     </xacro:kinect_camera>
+    <!-- Kinect -->
+    <!--xacro:include filename="$(find quadrotor_controller)/urdf/kinect_camera_viewfield.urdf.xacro" />
+    <xacro:kinect_camera01 name="camera01" parent="base_link">
+    <origin xyz="-1 0.0 0.3" rpy="0 0.2 0"/>
+    </xacro:kinect_camera01-->
 </robot>
